Commit message: edit joint type and add transmission tag

File: quadcopter/urdf/quad.urdf.xacro (robot description, xacro)
@@ -6,5 +6,7 @@
   <joint name="quad_joint" type="fixed">
     <!-- THe CoG of the quadcopter 7cm below of the quadcopter frame axis -->
-    <origin xyz="0 0 0" rpy="0 0 0"/>
+    <origin xyz="0 0 -0.07" rpy="0 0 0"/>
+    <axis xyz="0 0 1"/>
+    <limit upper="0.0" lower="3.14" effort="2" velocity="2.0"/>
     <parent link="map"/>
     <child link="quad_link"/>
@@ -15,5 +17,5 @@
       <origin xyz="0 0 0" rpy="0 0 0"/>
       <geometry>
-        <mesh filename="package://quad_sim/desc/meshes/quad.dae"/>
+	      <mesh filename="package://quad_sim/quadcopter/meshes/quad.obj"/>
       </geometry>
     </visual>
@@ -21,5 +23,5 @@
       <origin xyz="0 0 0" rpy="0 0 0"/>
       <geometry>
-        <mesh filename="package://quad_sim/desc/meshes/quad.stl"/>
+	      <mesh filename="package://quad_sim/quadcopter/meshes/quad.stl"/>
       </geometry>
     </collision>
@@ -30,4 +32,13 @@
     </inertial>
   </link>
+  <transmission name="trans1">
+	  <type>transmission_interface/SimpleTransmission</type>
+	  <joint name="quad_joint">
+		  <hardwareInterface>EffortJointInterface</hardwareInterface>
+	  </joint>
+	  <actuator>
+		  <hardwareInterface>EffortJointInterface</hardwareInterface>
+	  </actuator>
+  </transmission>
   <!-- xacro:include filename="world.xacro" -->
 </robot>
