Commit message: update quadcopter's mesh

File: quadcopter/urdf/frame.xacro (robot description, xacro)
@@ -11,5 +11,5 @@
         <origin xyz="0 0 0" rpy="0 0 0"/>
         <geometry>
-          <mesh filename="package://quad_sim/quadcopter/meshes/quad_frame.dae"/>
+          <mesh filename="package://quad_sim/quadcopter/meshes/quad_frame2.dae"/>
         </geometry>
       </visual>
@@ -17,5 +17,5 @@
         <origin xyz="0 0 0" rpy="0 0 0"/>
         <geometry>
-          <mesh filename="package://quad_sim/quadcopter/meshes/quad_frame.stl"/>
+          <mesh filename="package://quad_sim/quadcopter/meshes/quad_frame2.stl" scale="0.001 0.001 0.001"/>
         </geometry>
       </collision>

File: quadcopter/urdf/marker.xacro (robot description, xacro)
@@ -11,11 +11,11 @@
         <origin xyz="0 0 0" rpy="0 0 0"/>
         <geometry>
-          <mesh filename="package://quad_sim/quadcopter/meshes/marker_raw.dae"/>
+          <sphere radius="0.025"/>
         </geometry>
       </visual>
       <collision>
-        <origin xyz="0 0 9" rpy="0 0 0"/>
+        <origin xyz="0 0 0" rpy="0 0 0"/>
         <geometry>
-          <mesh filename="package://quad_sim/quadcopter/meshes/marker_raw.stl"/>
+          <sphere radius="0.025"/>
         </geometry>
       </collision>

File: quadcopter/urdf/quad_base.urdf.xacro (robot description, xacro)
@@ -49,20 +49,20 @@
   <!--Marker's Joints-->
   <joint name="marker1_joint" type="fixed">
-    <origin xyz="0.205 0.205 0.05" rpy="0 0 0"/>
+    <origin xyz="0.205 0.205 0.06" rpy="0 0 0"/>
     <parent link="frame_link"/>
     <child link="marker1_link"/>
   </joint>
   <joint name="marker2_joint" type="fixed">
-    <origin xyz="-0.205 0.205 0.05" rpy="0 0 0"/>
+    <origin xyz="-0.205 0.205 0.06" rpy="0 0 0"/>
     <parent link="frame_link"/>
     <child link="marker2_link"/>
   </joint>
   <joint name="marker3_joint" type="fixed">
-    <origin xyz="-0.205 -0.205 0.05" rpy="0 0 0"/>
+    <origin xyz="-0.205 -0.205 0.06" rpy="0 0 0"/>
     <parent link="frame_link"/>
     <child link="marker3_link"/>
   </joint>
   <joint name="marker4_joint" type="fixed">
-    <origin xyz="0.205 -0.205 0.05" rpy="0 0 0"/>
+    <origin xyz="0.205 -0.205 0.06" rpy="0 0 0"/>
     <parent link="frame_link"/>
     <child link="marker4_link"/>

File: quadcopter/urdf/rotor.xacro (robot description, xacro)
@@ -11,5 +11,5 @@
         <origin xyz="0 0 0" rpy="0 0 0"/>
         <geometry>
-          <mesh filename="package://quad_sim/quadcopter/meshes/quad_rotor.dae"/>
+          <mesh filename="package://quad_sim/quadcopter/meshes/quad_rotor.dae" scale="0.74359 0.74359 0"/>
         </geometry>
       </visual>
@@ -17,10 +17,10 @@
         <origin xyz="0 0 0" rpy="0 0 0"/>
         <geometry>
-          <mesh filename="package://quad_sim/quadcopter/meshes/quad_rotor.stl"/>
+          <mesh filename="package://quad_sim/quadcopter/meshes/quad_rotor.stl" scale="0.00074359 0.00074359 0.001"/>
         </geometry>
       </collision>
     </link>
   <gazebo reference="rotor_link">
-    <material>Gazebo/Gray</material>
+    <material>Gazebo/Grey</material>
   </gazebo>
   </xacro:macro>
