Commit message: edit the camera model

File: camera_sensor/tutorial/camera1.xacro (robot description, xacro)
@@ -2,45 +2,65 @@
 <robot xmlns:xacro="http://www.ros.org/wiki/xacro" name="camera1">
 	<link name="cam">
-		<static>true</static>
-		<visual name="cam_visual">
-			<origin xyz="-1 0 1" rpy="0 1 0"/>
+    <inertial>
+      <origin xyz="0 0 0" rpy="0 0 0"/>
+      <mass value="0.1"/>
+      <inertia ixx="0.000166667" ixy="0.0" ixz="0.0" iyy="0.000166667" iyz="0.0" izz="0.000166667"/>
+    </inertial>
+    <visual name="cam_visual">
+			<origin xyz="0 0 0" rpy="0 0 0"/>
 			<geometry>
-				<box>
-					<size>.1 .1 .1</size>
-				</box>
+				<box size=".1 .1 .1"/>
 			</geometry>
 		</visual>
-		<sensor name="cam_sensor" type="camera">
-			<update_rate>30.0</update_rate>
-			<camera>
-				<horizontal_fov>1.3962634</horizontal_fov>
-				<image>
-					<width>800</width>
-					<height>800</height>
-					<format>R8G8B8</format>
-				</image>
-				<clip>
-					<near>0.02</near>
-					<far>300</far>
-				</clip>
-				<noise>
-					<type>gaussian</type>
-					<mean>0.0</mean>
-					<stddev>0.0</stddev>
-				</noise>
-			</camera>
-			<plugin name="camera_controller" filename="libgazebo_rps_camera.so">
-				<cameraName>camera1</cameraName>
-				<imageTopicName>image_raw</imageTopicName>
-				<cameraInfoTopicName>camera_info</cameraInfoTopicName>
-				<frameName>cam_link</frameName>
-				<hackBaseline>0.0</hackBaseline>
-				<distortionK1>0.0</distortionK1>
-				<distortionK2>0.0</distortionK2>
-				<distortionK3>0.0</distortionK3>
-				<distortionT1>0.0</distortionT1>
-				<distortionT2>0.0</distortionT2>
-			</plugin>
-		</sensor>
+    <collision  name="cam_collision">
+			<origin xyz="0 0 0" rpy="0 0 0"/>
+			<geometry>
+        <box size=".1 .1 .1"/>
+			</geometry>
+		</collision>
 	</link>
-</robot>
+    <!-- camera -->
+  <gazebo>
+    <static>true</static>
+  </gazebo>
+  <gazebo reference="cam">
+    <static>true</static>
+    <sensor type="camera" name="camera1">
+      <update_rate>30.0</update_rate>
+      <camera name="nom">
+        <horizontal_fov>1.3962634</horizontal_fov>
+        <image>
+          <width>800</width>
+          <height>800</height>
+          <format>R8G8B8</format>
+        </image>
+        <clip>
+          <near>0.02</near>
+          <far>300</far>
+        </clip>
+        <noise>
+          <type>gaussian</type>
+          <!-- Noise is sampled independently per pixel on each frame.
+               That pixel's noise value is added to each of its color
+               channels, which at that point lie in the range [0,1]. -->
+          <mean>0.0</mean>
+          <stddev>0.007</stddev>
+        </noise>
+      </camera>
+      <plugin name="camera_controller" filename="libgazebo_ros_camera.so">
+        <alwaysOn>true</alwaysOn>
+        <updateRate>0.0</updateRate>
+        <cameraName>cam1</cameraName>
+        <imageTopicName>image_raw</imageTopicName>
+        <cameraInfoTopicName>cam1_info</cameraInfoTopicName>
+        <frameName>camera_link</frameName>
+        <hackBaseline>0.07</hackBaseline>
+        <distortionK1>0.0</distortionK1>
+        <distortionK2>0.0</distortionK2>
+        <distortionK3>0.0</distortionK3>
+        <distortionT1>0.0</distortionT1>
+        <distortionT2>0.0</distortionT2>
+      </plugin>
+    </sensor>
+  </gazebo>
+ </robot>
