Commit message: adding launch file to spawn quadcopter and camera1

File: camera_sensor/one_camera/camera1.xacro (robot description, xacro)
@@ -1,5 +1,5 @@
 <?xml version="1.0"?>
 <robot xmlns:xacro="http://www.ros.org/wiki/xacro" name="camera1">
-	<link name="cam">
+  <link name="cam">
     <inertial>
       <origin xyz="0 0 0" rpy="0 0 0"/>
@@ -20,10 +20,8 @@
 		</collision>
 	</link>
-    <!-- camera -->
   <gazebo>
     <static>true</static>
   </gazebo>
   <gazebo reference="cam">
-    <static>true</static>
     <sensor type="camera" name="camera1">
       <update_rate>30.0</update_rate>
@@ -41,7 +39,7 @@
         <noise>
           <type>gaussian</type>
-          <!-- Noise is sampled independently per pixel on each frame.
+          <!--Noise is sampled independently per pixel on each frame.
                That pixel's noise value is added to each of its color
-               channels, which at that point lie in the range [0,1]. -->
+               channels, which at that point lie in the range [0,1].-->
           <mean>0.0</mean>
           <stddev>0.007</stddev>

File: quadcopter/urdf/quad_base.urdf.xacro (robot description, xacro)
@@ -2,7 +2,7 @@
 <robot xmlns:xacro="http://www.ros.org/wiki/xacro" name="quadcopter">
   <!--Include Frame, Rotor, and Marker model -->
-  <xacro:include filename="$(find quad_sim)/quadcopter/urdf/frame.xacro"/>
-  <xacro:include filename="$(find quad_sim)/quadcopter/urdf/rotor.xacro"/>
-  <xacro:include filename="$(find quad_sim)/quadcopter/urdf/marker.xacro"/>
+  <xacro:include filename="$(find quad_sim)/quadcopter/urdf/base/frame.xacro"/>
+  <xacro:include filename="$(find quad_sim)/quadcopter/urdf/base/rotor.xacro"/>
+  <xacro:include filename="$(find quad_sim)/quadcopter/urdf/base/marker.xacro"/>
 	<!-- Quadcopter Description -->
 	<xacro:macro name="quad_base_macro">
